File: jtag-20pin-to-10pin.kicad_pcb (KiCad board)
At the start: 2 copper layers, 18.4 x 34.3 mm, 2 parts, among them P1 CONN_02X10, P2 CONN_02X05

Commit message: make it round
Routing:
- net VTref: track 13.5 -> 15.7 mm
- net TDI: track 13.4 -> 14.5 mm
Other:
- board size 18.4 x 34.3 mm -> 17.8 x 33 mm
- board text added: "https://bytewerk.org/"
Changed lines of the file:
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@@
     (links 16)
     (no_connects 0)
-    (area 134.544999 90.729999 153.110001 125.170001)
+    (area 134.544999 91.364999 152.475001 124.535001)
     (thickness 1.6)
-    (drawings 25)
-    (tracks 15)
+    (drawings 34)
+    (tracks 22)
     (zones 0)
     (modules 2)
@@
     )
   )
+  (gr_line (start 147.32 115.57) (end 147.32 123.19) (layer Edge.Cuts) (width 0.15))
+  (gr_line (start 147.32 92.71) (end 147.32 100.33) (layer Edge.Cuts) (width 0.15))
+  (gr_line (start 152.4 102.87) (end 152.4 113.03) (layer Edge.Cuts) (width 0.15))
+  (gr_line (start 148.59 101.6) (end 151.13 101.6) (layer Edge.Cuts) (width 0.15))
+  (gr_arc (start 151.13 102.87) (end 151.13 101.6) (angle 90) (layer Edge.Cuts) (width 0.15))
+  (gr_line (start 151.13 114.3) (end 148.59 114.3) (layer Edge.Cuts) (width 0.15))
+  (gr_arc (start 151.13 113.03) (end 152.4 113.03) (angle 90) (layer Edge.Cuts) (width 0.15))
+  (gr_arc (start 148.59 115.57) (end 147.32 115.57) (angle 90) (layer Edge.Cuts) (width 0.15))
+  (gr_arc (start 148.59 100.33) (end 148.59 101.6) (angle 90) (layer Edge.Cuts) (width 0.15))
+  (gr_arc (start 146.05 92.71) (end 146.05 91.44) (angle 90) (layer Edge.Cuts) (width 0.15))
+  (gr_arc (start 146.05 123.19) (end 147.32 123.19) (angle 90) (layer Edge.Cuts) (width 0.15))
+  (gr_arc (start 135.89 123.19) (end 135.89 124.46) (angle 90) (layer Edge.Cuts) (width 0.15))
+  (gr_arc (start 135.89 92.71) (end 134.62 92.71) (angle 90) (layer Edge.Cuts) (width 0.15))
+  (gr_line (start 135.89 124.46) (end 146.05 124.46) (layer Edge.Cuts) (width 0.15))
+  (gr_line (start 134.62 123.19) (end 134.62 92.71) (layer Edge.Cuts) (width 0.15))
+  (gr_line (start 135.89 91.44) (end 146.05 91.44) (layer Edge.Cuts) (width 0.15))
+  (gr_text https://bytewerk.org/ (at 145.542 107.95 90) (layer F.SilkS)
+    (effects (font (size 1.5 1.5) (thickness 0.3)))
+  )
   (gr_line (start 136.144 96.52) (end 137.16 96.52) (layer B.SilkS) (width 0.2))
   (gr_line (start 136.144 99.06) (end 137.16 99.06) (layer B.SilkS) (width 0.2))
@@
     (effects (font (size 1.2 1.2) (thickness 0.3)) (justify right mirror))
   )
-  (gr_line (start 146.05 90.805) (end 153.035 97.79) (layer Edge.Cuts) (width 0.15))
-  (gr_line (start 153.035 118.11) (end 146.05 125.095) (layer Edge.Cuts) (width 0.15))
-  (gr_line (start 134.62 125.095) (end 134.62 90.805) (layer Edge.Cuts) (width 0.15))
-  (gr_line (start 143.51 125.095) (end 134.62 125.095) (layer Edge.Cuts) (width 0.15))
-  (gr_line (start 146.05 125.095) (end 143.51 125.095) (layer Edge.Cuts) (width 0.15))
-  (gr_line (start 153.035 97.79) (end 153.035 118.11) (layer Edge.Cuts) (width 0.15))
-  (gr_line (start 143.51 90.805) (end 146.05 90.805) (layer Edge.Cuts) (width 0.15))
-  (gr_line (start 134.62 90.805) (end 143.51 90.805) (layer Edge.Cuts) (width 0.15))
-  (segment (start 140.97 119.38) (end 142.07 119.38) (width 0.25) (layer F.Cu) (net 1))
-  (segment (start 142.07 119.38) (end 150.495 110.955) (width 0.25) (layer F.Cu) (net 1))
-  (segment (start 150.495 110.955) (end 150.495 110.49) (width 0.25) (layer F.Cu) (net 1))
-  (segment (start 140.97 114.3) (end 142.849206 112.420794) (width 0.25) (layer B.Cu) (net 3))
-  (segment (start 142.849206 112.420794) (end 142.849206 109.028549) (width 0.25) (layer B.Cu) (net 3))
-  (segment (start 142.849206 109.028549) (end 145.197755 106.68) (width 0.25) (layer B.Cu) (net 3))
+  (segment (start 140.97 119.38) (end 142.299374 119.38) (width 0.25) (layer F.Cu) (net 1))
+  (segment (start 142.299374 119.38) (end 143.172465 118.506909) (width 0.25) (layer F.Cu) (net 1))
+  (segment (start 149.34 112.395) (end 150.495 111.24) (width 0.25) (layer F.Cu) (net 1))
+  (segment (start 143.172465 118.506909) (end 143.172465 114.951798) (width 0.25) (layer F.Cu) (net 1))
+  (segment (start 143.172465 114.951798) (end 145.729263 112.395) (width 0.25) (layer F.Cu) (net 1))
+  (segment (start 145.729263 112.395) (end 149.34 112.395) (width 0.25) (layer F.Cu) (net 1))
+  (segment (start 150.495 111.24) (end 150.495 110.49) (width 0.25) (layer F.Cu) (net 1))
+  (segment (start 140.97 114.3) (end 142.853162 114.3) (width 0.25) (layer B.Cu) (net 3))
+  (segment (start 144.160635 107.71712) (end 145.197755 106.68) (width 0.25) (layer B.Cu) (net 3))
+  (segment (start 142.853162 114.3) (end 144.160635 112.992527) (width 0.25) (layer B.Cu) (net 3))
+  (segment (start 144.160635 112.992527) (end 144.160635 107.71712) (width 0.25) (layer B.Cu) (net 3))
   (segment (start 145.197755 106.68) (end 149.225 106.68) (width 0.25) (layer B.Cu) (net 3))
   (segment (start 140.97 111.76) (end 143.524853 111.76) (width 0.25) (layer F.Cu) (net 4))
@@
   (segment (start 144.794853 110.49) (end 149.225 110.49) (width 0.25) (layer F.Cu) (net 4))
   (segment (start 149.225 109.22) (end 140.97 109.22) (width 0.25) (layer F.Cu) (net 5))
-  (segment (start 140.97 104.14) (end 144.78 107.95) (width 0.25) (layer F.Cu) (net 6))
-  (segment (start 144.78 107.95) (end 149.225 107.95) (width 0.25) (layer F.Cu) (net 6))
-  (segment (start 140.97 101.6) (end 144.78 105.41) (width 0.25) (layer F.Cu) (net 7))
-  (segment (start 144.78 105.41) (end 149.225 105.41) (width 0.25) (layer F.Cu) (net 7))
+  (segment (start 140.97 104.14) (end 143.117885 104.14) (width 0.25) (layer F.Cu) (net 6))
+  (segment (start 143.117885 104.14) (end 146.927885 107.95) (width 0.25) (layer F.Cu) (net 6))
+  (segment (start 146.927885 107.95) (end 149.225 107.95) (width 0.25) (layer F.Cu) (net 6))
+  (segment (start 142.875 101.6) (end 146.685 105.41) (width 0.25) (layer F.Cu) (net 7))
+  (segment (start 146.685 105.41) (end 149.225 105.41) (width 0.25) (layer F.Cu) (net 7))
+  (segment (start 140.97 101.6) (end 142.875 101.6) (width 0.25) (layer F.Cu) (net 7))
   (zone (net 2) (net_name GND) (layer B.Cu) (hatch edge 0.508)
     (connect_pads (clearance 0.2))
